File: iceglue.kicad_pcb (KiCad board)
At the start: 2 copper layers, 36 parts, among them J1 USB_OTG, J2 TEST_1P, J3 Conn_01x21, J4 Conn_01x21, J5 TEST_1P, SW1 SW_Push, U1 STM32F070F6P6, U2 ICE40UP5K-SG48, U3 LD1117S33TR_SOT223, U4 LD1117S12TR_SOT223

Commit message: lalalal
Parts:
- C1, C14, C15, C17, C4, C5, C8, C9, D2, JP1, R4: moved to B.Cu
- U3: footprint sot:SOT23 -> TO_SOT_Packages_SMD:SOT-223-3_TabPin2
- U4: footprint sot:SOT23 -> TO_SOT_Packages_SMD:SOT-223-3_TabPin2; moved to B.Cu
- moved R1 57.0 mm to (157.3, 149.6), turned to 180 degrees
- moved C11 48.4 mm to (152.4, 114.3), turned to 270 degrees
- moved D2 46.6 mm to (163.6, 147.3), turned to 180 degrees
- moved JP1 45.9 mm to (160.5, 117.3), turned to 180 degrees
- moved C2 45.0 mm to (159.5, 111.5), turned to 180 degrees
- moved R3 44.6 mm to (165.4, 152.4), turned to 90 degrees
- moved C1 39.9 mm to (160.0, 106.9), turned to 180 degrees
- moved R4 34.9 mm to (160.9, 137.8)
- moved R2 34.6 mm to (157.1, 119.0), turned to 90 degrees
- moved C8 34.3 mm to (158.5, 140.5), turned to 270 degrees
- moved C13 33.4 mm to (155.7, 128.4)
- moved C10 31.2 mm to (207.6, 147.9)
- moved C6 30.8 mm to (207.3, 142.3)
- moved C16 29.7 mm to (207.2, 145.2)
- moved C4 26.6 mm to (156.8, 134.4), turned to 270 degrees
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Connections:
- C14 pad 1: +3V3 -> +1V2
- J1 pad 4: (no net) -> Net-(J1-Pad4)
- J4 pad 11: /IO_27 -> /IO_25
- J4 pad 12: /IO_28 -> /IO_24
- J4 pad 13: /IO_29 -> /IO_23
- J4 pad 14: /IO_30 -> /IO_22
- J4 pad 15: /IO_31 -> /IO_21
- J4 pad 16: /IO_32 -> /IO_20
- J4 pad 17: /IO_33 -> /IO_19
- J4 pad 18: /IO_34 -> /IO_18
- J4 pad 2: /IO_18 -> /IO_34
- J4 pad 3: /IO_19 -> /IO_33
- J4 pad 4: /IO_20 -> /IO_32
- J4 pad 5: /IO_21 -> /IO_31
- J4 pad 6: /IO_22 -> /IO_30
- J4 pad 7: /IO_23 -> /IO_29
- J4 pad 8: /IO_24 -> /IO_28
- J4 pad 9: /IO_25 -> /IO_27
- U1 pad 10: (no net) -> Net-(U1-Pad10)
- U1 pad 14: (no net) -> Net-(U1-Pad14)
- U1 pad 19: (no net) -> Net-(U1-Pad19)
- U1 pad 2: (no net) -> Net-(U1-Pad2)
- U1 pad 3: (no net) -> Net-(U1-Pad3)
- U1 pad 6: (no net) -> Net-(U1-Pad6)
- U1 pad 7: (no net) -> Net-(U1-Pad7)
- U1 pad 8: (no net) -> Net-(U1-Pad8)
- U1 pad 9: (no net) -> Net-(U1-Pad9)
- U4 pad 2: +3V3 -> +1V2
Routing:
- net GND: track 0.00 -> 63.3 mm, vias 0 -> 2
- net /RESET: track 0.00 -> 50.3 mm, vias 0 -> 1
- net /SPI_SCK: track 0.00 -> 46.2 mm, vias 0 -> 1
- net /SPI_MISO: track 0.00 -> 43.9 mm, vias 0 -> 1
- net /SPI_MOSI: track 0.00 -> 42.0 mm, vias 0 -> 1
- net +3V3: track 0.00 -> 32.8 mm, vias 0 -> 2
- net /IO_0: track 0.00 -> 30.5 mm
- net /IO_34: track 0.00 -> 29.8 mm
- net /IO_1: track 0.00 -> 27.8 mm
- net /IO_33: track 0.00 -> 27.1 mm
- net /IO_2: track 0.00 -> 25.0 mm
- net /IO_32: track 0.00 -> 24.3 mm
- net /IO_BTN: track 0.00 -> 23.5 mm, vias 0 -> 2
- net /IO_3: track 0.00 -> 22.3 mm
- net +5V: track 0.00 -> 21.6 mm
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Other:
- board outline added: 23.6 x 55.1 mm
- net class io added: clearance 0.2, trace_width 0.25, via_dia 0.6, via_drill 0.3
- net class power added: clearance 0.2, trace_width 0.5, via_dia 0.6, via_drill 0.4

Commit message: fully layouted; ready to use ;)
Parts:
- removed R5: 10k, Resistors_SMD:R_0603_HandSoldering
- added J6: TEST_1P, Measurement_Points:Measurement_Point_Round-SMD-Pad_Small, B.Cu at (153.2, 111.0)
- C10, C13, C16, C6, C7, J2, J5: moved to B.Cu
- C17, D2: moved to F.Cu
- C3: value 0.1µ -> 1µ; moved to B.Cu
- J3, J4: value Conn_01x21 -> Conn_01x22; footprint Pin_Headers:Pin_Header_Straight_1x21_Pitch2.54mm -> Pin_Headers:Pin_Header_Straight_1x22_Pitch2.54mm; moved to B.Cu
- moved C3 53.6 mm to (153.9, 132.6), turned to 90 degrees
- moved C7 50.1 mm to (158.0, 140.5), turned to 270 degrees
- moved C16 44.4 mm to (162.9, 142.0), turned to 270 degrees
- moved C10 44.3 mm to (164.3, 138.2), turned to 90 degrees
- moved C6 42.7 mm to (165.1, 148.8)
- moved J2 33.6 mm to (154.2, 115.8)
- moved C12 32.5 mm to (160.3, 131.6)
- moved J5 30.2 mm to (155.2, 109.0)
- moved U4 27.3 mm to (157.6, 155.2), turned to 0 degrees
- moved C13 24.5 mm to (152.4, 152.7), turned to 270 degrees
- moved C14 22.9 mm to (152.4, 156.5), turned to 270 degrees
- moved C11 12.4 mm to (161.8, 122.4), turned to 180 degrees
- moved U3 4.98 mm to (159.8, 127.0), turned to 180 degrees
- moved C17 3.52 mm to (166.3, 148.1), turned to 0 degrees
- moved R3 2.18 mm to (164.1, 154.2)
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Connections:
- J1 pad 4: Net-(J1-Pad4) -> (no net)
- U1 pad 10: Net-(U1-Pad10) -> (no net)
- U1 pad 14: Net-(U1-Pad14) -> (no net)
- U1 pad 19: Net-(U1-Pad19) -> (no net)
- U1 pad 2: Net-(U1-Pad2) -> (no net)
- U1 pad 3: Net-(U1-Pad3) -> (no net)
- U1 pad 6: Net-(U1-Pad6) -> (no net)
- U1 pad 7: Net-(U1-Pad7) -> (no net)
- U1 pad 8: Net-(U1-Pad8) -> (no net)
- U1 pad 9: Net-(U1-Pad9) -> (no net)
Routing:
- net GND: track 63.3 -> 244.6 mm, vias 2 -> 8
- net +5V: track 21.6 -> 156.5 mm, vias 0 -> 5
- net +3V3: track 32.8 -> 117.3 mm, vias 2 -> 7
- net +1V2: track 3.66 -> 51.0 mm, vias 0 -> 2
- net /IO_LED: track 0.00 -> 32.0 mm, vias 0 -> 2
- net Net-(JP2-Pad2): track 17.3 -> 7.28 mm
- net /SPI_MISO: track 43.9 -> 52.9 mm
- net /IO_BTN: track 23.5 -> 30.5 mm
- net /SPI_MOSI: track 42.0 -> 48.6 mm
- net Net-(C15-Pad1): track 3.62 -> 9.22 mm, vias 0 -> 1
- net /SPI_SCK: track 46.2 -> 51.1 mm, vias 1 -> 2
- net +2V5: track 0.00 -> 4.90 mm
- net /IO_29: track 12.1 -> 16.1 mm
- net /IO_28: track 18.1 -> 14.6 mm
- net /IO_19: track 9.18 -> 12.3 mm
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Other:
- board size 23.6 x 55.1 mm -> 23.6 x 57.7 mm

Commit message: minor corrections
Routing:
- net /IO_2: track 26.6 -> 25.0 mm
- net /IO_4: track 21.1 -> 19.5 mm
- net /IO_3: track 23.8 -> 22.3 mm
- net /IO_1: track 29.3 -> 27.8 mm
- net /IO_0: track 32.0 -> 30.5 mm
- net /IO_9: track 14.0 -> 12.7 mm
- net /IO_10: track 12.1 -> 10.7 mm
- net /IO_11: track 10.1 -> 8.76 mm
- net /RESET: track 49.3 -> 48.0 mm
- net /IO_5: track 17.7 -> 16.8 mm
- net +5V: track 156.5 -> 155.7 mm
- net /IO_19: track 12.3 -> 11.7 mm
- net /SPI_SCK: track 51.1 -> 50.9 mm, vias 2 -> 1
